File: esp-stack-mini.sch (EAGLE design)
At the start: 61 parts, among them IC1 FT232RL, Q1 BSS138, Q2 AO3401, Q3 S8050, Q4 S8050, U1 TPS737XX, U2 MCP73831

Commit message: progress
Parts:
- R17: value 470 -> 220k
- R18: value 470 -> 51k
- R19: value 4k7 -> 9k1
Connections:
- net D0: now also H5.D0, MODE.2, Q3.P$2, R19.1; no longer Q3.P$3
- net D15: no longer H5.D15, MODE.2, R19.1
- net N$15: now also Q4.P$3; no longer Q4.P$2
- net N$16: now also Q3.P$3; no longer Q3.P$2
- net RST: now also Q4.P$2; no longer Q4.P$3
- net V+: now also D1.VDD, D2.VDD, D3.VDD, D4.VDD, JP2.3, R8.2
- net VBUS: no longer D1.VDD, D2.VDD, D3.VDD, D4.VDD, JP2.3, R8.2
Changed lines of the file:
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@@
 <part name="SJ1" library="jumper" deviceset="SJ" device="" value="SLEEP"/>
 <part name="H4" library="ESPStack-mini" deviceset="ESP-BOARD" device=""/>
-<part name="R17" library="resistor" deviceset="R-EU_" device="R0805" value="470"/>
-<part name="R18" library="resistor" deviceset="R-EU_" device="R0805" value="470"/>
+<part name="R17" library="resistor" deviceset="R-EU_" device="R0805" value="220k"/>
+<part name="R18" library="resistor" deviceset="R-EU_" device="R0805" value="51k"/>
 <part name="GND16" library="supply1" deviceset="GND" device=""/>
 <part name="HX711" library="SparkFun-Connectors" deviceset="M04" device="NO_SILK_ALL_ROUND"/>
@@
 <part name="DHT11/22" library="SparkFun-Connectors" deviceset="M04" device="NO_SILK_ALL_ROUND"/>
 <part name="1WIRE" library="SparkFun-Connectors" deviceset="M03" device="PTH"/>
-<part name="R19" library="resistor" deviceset="R-EU_" device="R0805" value="4k7"/>
+<part name="R19" library="resistor" deviceset="R-EU_" device="R0805" value="9k1"/>
 <part name="MODE" library="SparkFun-Retired" deviceset="SOLDERJUMPER_2WAY" device="T"/>
 <part name="H6" library="ESPStack-mini" deviceset="ESP-BOARD" device=""/>
@@
 </segment>
 <segment>
-<pinref part="Q4" gate="G$1" pin="P$3"/>
+<pinref part="Q4" gate="G$1" pin="P$2"/>
 <wire x1="134.62" y1="213.36" x2="134.62" y2="210.82" width="0.1524" layer="91"/>
 <label x="134.62" y="210.82" size="1.778" layer="95" xref="yes"/>
@@
 <wire x1="116.84" y1="152.4" x2="116.84" y2="157.48" width="0.1524" layer="91"/>
 <label x="116.84" y="152.4" size="1.778" layer="95" xref="yes"/>
+</segment>
+<segment>
+<pinref part="R8" gate="G$1" pin="2"/>
+<wire x1="353.06" y1="45.72" x2="353.06" y2="48.26" width="0.1524" layer="91"/>
+<label x="353.06" y="48.26" size="1.4224" layer="95" rot="R90" xref="yes"/>
+</segment>
+<segment>
+<pinref part="D1" gate="G$1" pin="VDD"/>
+<wire x1="421.64" y1="5.08" x2="421.64" y2="10.16" width="0.1524" layer="91"/>
+<wire x1="421.64" y1="10.16" x2="393.7" y2="10.16" width="0.1524" layer="91"/>
+<wire x1="393.7" y1="10.16" x2="365.76" y2="10.16" width="0.1524" layer="91"/>
+<wire x1="365.76" y1="10.16" x2="335.28" y2="10.16" width="0.1524" layer="91"/>
+<wire x1="335.28" y1="10.16" x2="320.04" y2="10.16" width="0.1524" layer="91"/>
+<wire x1="320.04" y1="10.16" x2="320.04" y2="0" width="0.1524" layer="91"/>
+<label x="421.64" y="10.16" size="1.778" layer="95" rot="R90" xref="yes"/>
+<pinref part="JP2" gate="G$1" pin="3"/>
+<pinref part="D4" gate="G$1" pin="VDD"/>
+<wire x1="337.82" y1="5.08" x2="335.28" y2="5.08" width="0.1524" layer="91"/>
+<wire x1="335.28" y1="5.08" x2="335.28" y2="10.16" width="0.1524" layer="91"/>
+<junction x="335.28" y="10.16"/>
+<pinref part="D3" gate="G$1" pin="VDD"/>
+<wire x1="365.76" y1="5.08" x2="365.76" y2="10.16" width="0.1524" layer="91"/>
+<junction x="365.76" y="10.16"/>
+<pinref part="D2" gate="G$1" pin="VDD"/>
+<wire x1="393.7" y1="5.08" x2="393.7" y2="10.16" width="0.1524" layer="91"/>
+<junction x="393.7" y="10.16"/>
 </segment>
 </net>
@@
 </segment>
 <segment>
-<pinref part="MODE" gate="G$1" pin="2"/>
-<wire x1="396.24" y1="175.26" x2="393.7" y2="175.26" width="0.1524" layer="91"/>
-<label x="393.7" y="175.26" size="1.778" layer="95" rot="R180" xref="yes"/>
-</segment>
-<segment>
-<pinref part="R19" gate="G$1" pin="1"/>
-<wire x1="401.32" y1="142.24" x2="401.32" y2="134.62" width="0.1524" layer="91"/>
-<label x="401.32" y="134.62" size="1.778" layer="95" xref="yes"/>
-</segment>
-<segment>
-<pinref part="H5" gate="G$1" pin="D15"/>
-<wire x1="403.86" y1="218.44" x2="408.94" y2="218.44" width="0.1524" layer="91"/>
-<label x="408.94" y="218.44" size="1.778" layer="95" xref="yes"/>
-</segment>
-<segment>
 <pinref part="H6" gate="G$1" pin="D15"/>
 <wire x1="520.7" y1="205.74" x2="523.24" y2="205.74" width="0.1524" layer="91"/>
@@
 </segment>
 <segment>
-<pinref part="Q3" gate="G$1" pin="P$3"/>
+<pinref part="Q3" gate="G$1" pin="P$2"/>
 <wire x1="134.62" y1="241.3" x2="134.62" y2="243.84" width="0.1524" layer="91"/>
 <label x="134.62" y="243.84" size="1.778" layer="95" xref="yes"/>
@@
 <label x="586.74" y="210.82" size="1.778" layer="95" xref="yes"/>
 </segment>
+<segment>
+<pinref part="MODE" gate="G$1" pin="2"/>
+<wire x1="396.24" y1="175.26" x2="393.7" y2="175.26" width="0.1524" layer="91"/>
+<label x="393.7" y="175.26" size="1.778" layer="95" rot="R180" xref="yes"/>
+</segment>
+<segment>
+<pinref part="R19" gate="G$1" pin="1"/>
+<wire x1="401.32" y1="142.24" x2="401.32" y2="134.62" width="0.1524" layer="91"/>
+<label x="401.32" y="134.62" size="1.778" layer="95" xref="yes"/>
+</segment>
+<segment>
+<pinref part="H5" gate="G$1" pin="D0"/>
+<wire x1="403.86" y1="223.52" x2="406.4" y2="223.52" width="0.1524" layer="91"/>
+<label x="406.4" y="223.52" size="1.778" layer="95" xref="yes"/>
+</segment>
 </net>
 <net name="D4" class="0">
@@
 <pinref part="H1" gate="G$1" pin="VBUS"/>
 <wire x1="172.72" y1="66.04" x2="170.18" y2="66.04" width="0.1524" layer="91"/>
-</segment>
-<segment>
-<pinref part="R8" gate="G$1" pin="2"/>
-<wire x1="353.06" y1="45.72" x2="353.06" y2="48.26" width="0.1524" layer="91"/>
-<label x="353.06" y="48.26" size="1.4224" layer="95" rot="R90" xref="yes"/>
-</segment>
-<segment>
-<pinref part="D1" gate="G$1" pin="VDD"/>
-<wire x1="421.64" y1="5.08" x2="421.64" y2="10.16" width="0.1524" layer="91"/>
-<wire x1="421.64" y1="10.16" x2="393.7" y2="10.16" width="0.1524" layer="91"/>
-<wire x1="393.7" y1="10.16" x2="365.76" y2="10.16" width="0.1524" layer="91"/>
-<wire x1="365.76" y1="10.16" x2="335.28" y2="10.16" width="0.1524" layer="91"/>
-<wire x1="335.28" y1="10.16" x2="320.04" y2="10.16" width="0.1524" layer="91"/>
-<wire x1="320.04" y1="10.16" x2="320.04" y2="0" width="0.1524" layer="91"/>
-<label x="421.64" y="10.16" size="1.778" layer="95" rot="R90" xref="yes"/>
-<pinref part="JP2" gate="G$1" pin="3"/>
-<pinref part="D4" gate="G$1" pin="VDD"/>
-<wire x1="337.82" y1="5.08" x2="335.28" y2="5.08" width="0.1524" layer="91"/>
-<wire x1="335.28" y1="5.08" x2="335.28" y2="10.16" width="0.1524" layer="91"/>
-<junction x="335.28" y="10.16"/>
-<pinref part="D3" gate="G$1" pin="VDD"/>
-<wire x1="365.76" y1="5.08" x2="365.76" y2="10.16" width="0.1524" layer="91"/>
-<junction x="365.76" y="10.16"/>
-<pinref part="D2" gate="G$1" pin="VDD"/>
-<wire x1="393.7" y1="5.08" x2="393.7" y2="10.16" width="0.1524" layer="91"/>
-<junction x="393.7" y="10.16"/>
 </segment>
 <segment>
@@
 <pinref part="R15" gate="G$1" pin="2"/>
 <wire x1="99.06" y1="236.22" x2="101.6" y2="236.22" width="0.1524" layer="91"/>
-<pinref part="Q4" gate="G$1" pin="P$2"/>
+<pinref part="Q4" gate="G$1" pin="P$3"/>
 <wire x1="101.6" y1="236.22" x2="111.76" y2="236.22" width="0.1524" layer="91"/>
 <wire x1="134.62" y1="223.52" x2="101.6" y2="223.52" width="0.1524" layer="91"/>
@@
 <wire x1="104.14" y1="218.44" x2="104.14" y2="228.6" width="0.1524" layer="91"/>
 <junction x="104.14" y="218.44"/>
-<pinref part="Q3" gate="G$1" pin="P$2"/>
+<pinref part="Q3" gate="G$1" pin="P$3"/>
 <wire x1="104.14" y1="228.6" x2="134.62" y2="228.6" width="0.1524" layer="91"/>
 <wire x1="134.62" y1="228.6" x2="134.62" y2="231.14" width="0.1524" layer="91"/>

Commit message: wip
Parts:
- removed 1WIRE: (no value), SparkFun-Connectors:M03PTH
- removed B1, B2: (no value), ESPStack-mini:SKSCLDE010
- removed D7: TX, diodes_gen:DIODE_SMDD0805
- removed D8: RX, diodes_gen:DIODE_SMDD0805
- removed J1: (no value), SparkFun-Connectors:JST_2MM_MALE
- removed R12, R13: 10k, resistor:R-EU_R0805
- added 1WIRE@1, 1WIRE@2: (no value), SparkFun-Connectors:M031X03_NO_SILK
- added BATT: (no value), SparkFun-Connectors:M021X02_NO_SILK
- added JP4: USB-A-H, SparkFun-Connectors:USB-A-H
- added JP5, JP6: (no value), SparkFun-Connectors:M14
- added POWER, SKIP: (no value), jumper:SJ
- added U$2, U$3: POGO-PAD, ESPStack-mini:POGO-PAD
- added USB_BREAKOUT, USB_BREAKOUT1: (no value), SparkFun-Connectors:M04NO_SILK_ALL_ROUND
- JP2: device SparkFun-Connectors:M03PTH -> SparkFun-Connectors:M031X03_NO_SILK
- R19: value 9k1 -> 4k7*
- R6: value 10k -> 470
- renumbered CHARGING to CHARG, MODE to DHT-MODE-1WIRE
Connections:
- removed net S1: H1.S, H6.S, H7.S, H8.S
- new net N$40: H6.D0, JP5.5
- new net N$52: H6.D2, JP5.6
- new net N$58: H6.D15, JP5.7
- new net N$65: H6.RST, JP6.14
- new net N$66: H6.ADC, JP6.13
- new net N$67: H6.EN, JP6.12
- new net N$68: H6.D16, JP6.11
- new net N$69: H6.D14, JP6.10
- new net N$70: H6.D12, JP6.9
- new net N$71: H6.D13, JP6.8
- new net NEOPIXEL_EXTERNAL: D4.DOUT, JP2.2, SKIP.2
- new net NEOPIXEL_VCC: D1.VDD, D2.VDD, D3.VDD, D4.VDD, JP2.3, POWER.1, R8.2
- new net VBAT: H6.VBATT, JP5.13
- net 1WIRE: now also 1WIRE@1.2, 1WIRE@2.2; no longer 1WIRE.2
- net 3V3: now also 1WIRE@1.1, 1WIRE@2.1, C2.+, H6.3V3@1, H6.3V3@2, H8.3V3@1, JP5.8, JP6.7; no longer 1WIRE.1, C1.+, D7.A, D8.A, R6.2
- net ADC: no longer H6.ADC, H8.ADC
- net CS0: now also H6.CS0, JP6.3
- net D+: now also JP4.D+, U$3.P$1, USB_BREAKOUT.2, USB_BREAKOUT1.2
- net D-: now also JP4.D-, U$2.P$1, USB_BREAKOUT.3, USB_BREAKOUT1.3
- net D0: no longer B2.1, H6.D0
- net D10: no longer H1.D10, H6.D10, H7.D10, H8.D10
- net D12: now also H5.D12; no longer H6.D12, H8.D12
- net D13: now also H5.D13; no longer H6.D13, H8.D13
- net D14: now also H5.D14; no longer H6.D14, H8.D14
- net D15: now also H5.D15; no longer H6.D15, H8.D15
- net D16: now also H5.D16; no longer H6.D16, H8.D16
- net D2: now also H5.D2; no longer B1.2, H6.D2, H8.D2, R6.1
- net D4: now also H5.D4; no longer H6.D4, H8.D4
- net D5: now also H5.D5; no longer H6.D5, H8.D5
- net D9: no longer H1.D9, H6.D9, H7.D9, H8.D9
- net GND: now also 1WIRE@1.3, 1WIRE@2.3, BATT.2, H6.GND@1, H6.GND@2, JP4.GND, JP5.14, JP5.9, JP6.1, JP6.2, JP6.6, USB_BREAKOUT.1, USB_BREAKOUT1.1; no longer 1WIRE.3, B1.4, B2.3, J1.-
- net MISO: now also H6.MISO, JP6.4
- net MOSI: now also H6.MOSI, JP6.5
- net N$17: now also H6.TX, JP5.1; no longer IC1.CBUS0, R12.2
- net N$18: now also H6.RX, JP5.2; no longer IC1.CBUS1, R13.2
- net N$19: now also H6.D5, JP5.3; no longer D7.K, R12.1
- net N$20: now also H6.D4, JP5.4; no longer D8.K, R13.1
- net N$4: now also IC1.RXD, R6.2; no longer D4.DOUT, JP2.2
- net NEOPIXEL: now also SKIP.1
- net RST: now also H8.RST
- net RX: now also H8.RX
- net SCLK: now also H6.SCLK, JP5.10
- net TX: now also H8.TX, R6.1; no longer IC1.RXD
- net V+: now also C1.+, H6.V+, JP5.11, POWER.2; no longer C2.+, D1.VDD, D2.VDD, D3.VDD, D4.VDD, JP2.3, R8.2
- net VBATT: now also BATT.1; no longer J1.+
- net VBUS: now also H6.VBUS, H8.VBUS, JP4.VBUS, JP5.12, USB_BREAKOUT.4, USB_BREAKOUT1.4
Other:
- moved on the sheet: BOOT, C1, C2, C5, IC1, Q3, Q4, R14, R15, R16, R6, U1
